Commit message: adding inertia values to link in urdf

File: examples/models/franka_description/robots/panda/franka2.urdf (robot description, URDF)
Before this commit: robot pandas, 41 links, 40 joints
Links:
- link camera_bottom_screw_frame: mass None -> 0.0
- link camera_color_frame: mass None -> 0.0
- link camera_color_optical_frame: mass None -> 0.0
- link camera_depth_frame: mass None -> 0.0
- link camera_infra1_frame: mass None -> 0.0
- link camera_infra1_optical_frame: mass None -> 0.0
- link camera_infra2_frame: mass None -> 0.0
- link camera_infra2_optical_frame: mass None -> 0.0
- link panda2_hand_sc: mass None -> 0.0
- link panda2_hand_tcp: mass None -> 0.0
- link panda2_link0_sc: mass None -> 0.0
- link panda2_link1_sc: mass None -> 0.0
- link panda2_link2_sc: mass None -> 0.0
- link panda2_link3_sc: mass None -> 0.0
- link panda2_link4_sc: mass None -> 0.0
- link panda2_link5_sc: mass None -> 0.0
- link panda2_link6_sc: mass None -> 0.0
- link panda2_link7_sc: mass None -> 0.0
- link panda2_link8: mass None -> 0.0
- link panda2_ref_camera_link: mass None -> 0.0
- link world: mass None -> 0.0

Commit message: changing the fingers by balls in the urdf

File: examples/models/franka_description/robots/panda/franka2.urdf (robot description, URDF)
Before this commit: robot pandas, 41 links, 40 joints
Links:
- link panda2_leftfinger: geometry collision sphere radius=0.03
- link panda2_rightfinger: geometry collision sphere radius=0.03

Commit message: changes in syntax in the code

File: examples/models/franka_description/robots/panda/franka2.urdf (robot description, URDF)
Before this commit: robot pandas, 41 links, 40 joints
Links:
- link camera_depth_optical_frame: mass None -> 0.0
