Commit message: clean the scene

File: examples/models/urdf/franka2.urdf (robot description, URDF)
Before this commit: robot pandas, 41 links, 40 joints
Links:
- removed link panda1_box
- removed link pedestal
- removed link wall_link_1
- removed link wall_link_2
- removed link wall_link_3
- link support_link: geometry collision box size=1.703 0.803 0.76; visual box size=1.703 0.803 0.76
Joints:
- removed joint panda1_box_joint
- removed joint pedestal_joint
- removed joint wall_joint_1
- removed joint wall_joint_2
- removed joint wall_joint_3
